File: kicad/Solar_Tracking_Board.kicad_pcb (KiCad board)
At the start: 2 copper layers, 53 x 68 mm, 23 parts, among them J1 Barrel_Jack, J10 Conn_01x03, J11 Conn_01x02_Female, J12 Conn_01x03, J13 Conn_01x02_Female, J14 MOUNTING_HOLE, J15 MOUNTING_HOLE, J16 MOUNTING_HOLE, J17 MOUNTING_HOLE, J2 Conn_02x03_Odd_Even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

Commit message: added gerbers
Parts:
- J11, J13: footprint Connectors_Molex:Molex_NanoFit_1x02x2.50mm_Straight -> Pin_Headers:Pin_Header_Straight_1x02_Pitch2.54mm
- moved J11 3.41 mm to (134.1, 76.2)
- moved J13 1.21 mm to (139.7, 76.2)
Connections:
- ICSP1 pad 1: (no net) -> Net-(ICSP1-Pad1)
- ICSP1 pad 2: (no net) -> Net-(ICSP1-Pad2)
- ICSP1 pad 3: (no net) -> Net-(ICSP1-Pad3)
- ICSP1 pad 4: (no net) -> Net-(ICSP1-Pad4)
- ICSP1 pad 5: (no net) -> Net-(ICSP1-Pad5)
- ICSP1 pad 6: (no net) -> Net-(ICSP1-Pad6)
- J1 pad 3: (no net) -> Net-(J1-Pad3)
- J3 pad 1: (no net) -> A0
- J4 pad 1: (no net) -> Net-(J4-Pad1)
- J4 pad 2: (no net) -> IOREF
- J4 pad 3: (no net) -> RESET
- J4 pad 4: (no net) -> +3V3
- J7 pad 1: (no net) -> SCL
- J7 pad 10: (no net) -> 8
- J7 pad 2: (no net) -> SDA
- J7 pad 3: (no net) -> AREF
- J7 pad 5: (no net) -> 13
- J7 pad 6: (no net) -> 12
- J7 pad 7: (no net) -> 11
- J7 pad 8: (no net) -> 10
- J7 pad 9: (no net) -> 9
- J8 pad 1: (no net) -> 7
- J8 pad 4: (no net) -> 4
- J8 pad 5: (no net) -> 3
- J8 pad 6: (no net) -> 2
- J8 pad 7: (no net) -> 1
- J8 pad 8: (no net) -> 0
Routing:
- net A5: track 0.00 -> 11.1 mm
- net Servo_PWR: track 37.4 -> 42.2 mm
- net SolarPWR_IN: track 9.75 -> 5.59 mm
