File: kicad/Solar_Tracking_Board.sch (KiCad schematic (older format))
At the start: 23 parts, among them J1 MOUNTING_HOLE, J10 MOUNTING_HOLE, J11 Conn_01x02_Female, J12 Conn_01x02_Female, J13 MOUNTING_HOLE, J14 Conn_01x08, J15 Conn_01x10, J16 Conn_01x06, J17 Conn_01x08, J18 Conn_02x03_Odd_Even, J2 Barrel_Jack, J3 Screw_Terminal_01x02, J4 Screw_Terminal_01x02, J5 Screw_Terminal_01x02, J6 MOUNTING_HOLE, J7 Conn_02x03_Odd_Even, J8 Conn_01x03, J9 Conn_01x03

Commit message: schematic footprints added
Parts:
- J11: footprint (none) -> Connectors_Molex:Molex_NanoFit_1x02x2.50mm_Straight
- J12: footprint (none) -> Connectors_Molex:Molex_NanoFit_1x02x2.50mm_Straight; P# (none) -> 105309-1102
- J3, J4, J5: footprint (none) -> TerminalBlock:TerminalBlock_bornier-2_P5.08mm
- RV1: footprint (none) -> Pin_Headers:Pin_Header_Straight_1x03_Pitch2.54mm
Changed lines of the file:
@@
 F 0 "J3" H 3700 1900 50  0000 C CNN
 F 1 "Screw_Terminal_01x02" H 3700 1600 50  0000 C CNN
-F 2 "" H 3700 1800 50  0001 C CNN
+F 2 "TerminalBlock:TerminalBlock_bornier-2_P5.08mm" H 3700 1800 50  0001 C CNN
 F 3 "" H 3700 1800 50  0001 C CNN
 	1    3700 1800
@@
 F 0 "J4" H 4650 1900 50  0000 C CNN
 F 1 "Screw_Terminal_01x02" H 4650 1600 50  0000 C CNN
-F 2 "" H 4650 1800 50  0001 C CNN
+F 2 "TerminalBlock:TerminalBlock_bornier-2_P5.08mm" H 4650 1800 50  0001 C CNN
 F 3 "" H 4650 1800 50  0001 C CNN
 	1    4650 1800
@@
 F 0 "J5" H 5650 1900 50  0000 C CNN
 F 1 "Screw_Terminal_01x02" H 5650 1600 50  0000 C CNN
-F 2 "" H 5650 1800 50  0001 C CNN
+F 2 "TerminalBlock:TerminalBlock_bornier-2_P5.08mm" H 5650 1800 50  0001 C CNN
 F 3 "" H 5650 1800 50  0001 C CNN
 	1    5650 1800
@@
 F 0 "J11" H 6150 3400 50  0000 C CNN
 F 1 "Conn_01x02_Female" H 6150 3100 50  0000 C CNN
-F 2 "" H 6150 3300 50  0001 C CNN
+F 2 "Connectors_Molex:Molex_NanoFit_1x02x2.50mm_Straight" H 6150 3300 50  0001 C CNN
 F 3 "" H 6150 3300 50  0001 C CNN
 	1    6150 3300
@@
 F 0 "J12" H 7200 3400 50  0000 C CNN
 F 1 "Conn_01x02_Female" H 7200 3100 50  0000 C CNN
-F 2 "" H 7200 3300 50  0001 C CNN
+F 2 "Connectors_Molex:Molex_NanoFit_1x02x2.50mm_Straight" H 7200 3300 50  0001 C CNN
 F 3 "" H 7200 3300 50  0001 C CNN
+F 4 "105309-1102" H 7200 3300 60  0001 C CNN "P#"
 	1    7200 3300
 	1    0    0    -1
@@
 F 0 "RV1" V 3025 6000 50  0000 C CNN
 F 1 "POT" V 3100 6000 50  0000 C CNN
-F 2 "" H 3200 6000 50  0001 C CNN
+F 2 "Pin_Headers:Pin_Header_Straight_1x03_Pitch2.54mm" H 3200 6000 50  0001 C CNN
 F 3 "" H 3200 6000 50  0001 C CNN
 	1    3200 6000

Commit message: schematic done
Parts:
- ICSP: renamed from J18; value Conn_02x03_Odd_Even -> Stack-Header_02x03_Odd_Even
- J14, J17: value Conn_01x08 -> Stack-Header_01x08
- J15: value Conn_01x10 -> Stack-Header_01x10
- J16: value Conn_01x06 -> Stack-Header_01x06
- R1, R2, R3, R4: value R -> 10k
Connections:
- net Barrel_PWR: now reaches J2.1
- net Barrel_PWR: now also J7.5 (Pin_5)
- net GND: now reaches J2.2
- net GND: now also J1.1, J10.1, J11.2 (Pin_2), J12.2 (Pin_2), J13.1, J14.6 (Pin_6), J14.7 (Pin_7), J15.4 (Pin_4), J3.1 (Pin_1), J6.1, J8.3 (Pin_3), J9.3 (Pin_3), R1.2, R2.2, R3.2, R4.2, RV1.3
- net +5V: now reaches J3.2 (Pin_2)
- net +5V: now also J14.5 (Pin_5), J7.1 (Pin_1), RV1.1
- net A1: now reaches J4.1 (Pin_1)
- net A1: now also J16.2 (Pin_2), R2.1
- net A2: now reaches J4.2 (Pin_2)
- net A2: now also J16.3 (Pin_3), R1.1
- net A3: now reaches J5.1 (Pin_1)
- net A3: now also J16.4 (Pin_4), R4.1
- net A4: now reaches J5.2 (Pin_2)
- net A4: now also J16.5 (Pin_5), R3.1
- net Servo_PWR: now reaches J7.2 (Pin_2)
- net Servo_PWR: now also J7.4 (Pin_4), J7.6 (Pin_6), J8.2 (Pin_2), J9.2 (Pin_2)
- net Vin: now reaches J7.3 (Pin_3)
- net Vin: now also J14.8 (Pin_8)
- net 6: now reaches J9.1 (Pin_1)
- net 6: now also J17.2 (Pin_2)
- net 5: now reaches J8.1 (Pin_1)
- net 5: now also J17.3 (Pin_3)
- net SCL: now reaches J15.1 (Pin_1)
- net 8: now reaches J15.10 (Pin_10)
- net SDA: now reaches J15.2 (Pin_2)
- net AREF: now reaches J15.3 (Pin_3)
- net 13: now reaches J15.5 (Pin_5)
- net 12: now reaches J15.6 (Pin_6)
- net 11: now reaches J15.7 (Pin_7)
- net 10: now reaches J15.8 (Pin_8)
- net 9: now reaches J15.9 (Pin_9)
- net 7: now reaches J17.1 (Pin_1)
- net 4: now reaches J17.4 (Pin_4)
- net 3: now reaches J17.5 (Pin_5)
- net 2: now reaches J17.6 (Pin_6)
- net 1: now reaches J17.7 (Pin_7)
- net 0: now reaches J17.8 (Pin_8)
- net IOREF: now reaches J14.2 (Pin_2)
- net RESET: now reaches J14.3 (Pin_3)
- net +3V3: now reaches J14.4 (Pin_4)
- net A0: now reaches J16.1 (Pin_1)
- net A5: now reaches J16.6 (Pin_6)
- net A5: now also RV1.2
- net SolarPWR_IN: now reaches J11.1 (Pin_1)
- net SolarPWR_OUT: now reaches J12.1 (Pin_1)
- no-connect marks 0 -> 8
Other:
- moved on the sheet: ICSP, J11, J12, J14, J15, J16, J17, J7, J8, J9, R1, R2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

Commit message: layout started
Parts:
- J16: renamed from J10; footprint Mounting_Holes:MountingHole_3.2mm_M3 -> Mounting_Holes:MountingHole_3.2mm_M3_Pad
- J4: renamed from J14; footprint Socket_Strips:Socket_Strip_Angled_1x08_Pitch2.54mm -> Pin_Headers:Pin_Header_Straight_1x08_Pitch2.54mm
- renumbered ICSP to ICSP1, J2 to J1, J9 to J10, J8 to J12, J12 to J13, J1 to J14, J6 to J15, J13 to J17, J7 to J2, J16 to J3, J3 to J5, J4 to J6, J15 to J7, J17 to J8, J5 to J9
Other:
- note added: "1"
- note added: "Arduino Shield for Solar Tracking"
- moved on the sheet: ICSP1, J1, J10, J11, J12, J13, J14, J15, J16, J17, J2, J3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

Commit message: Board Rev1 finsihed
Connections:
- net SolarPWR_OUT is gone; now on net SolarPWR_IN: J13.1 (Pin_1)
Changed lines of the file:
@@
 Text GLabel 6800 3650 0    39   Input ~ 0
 SolarPWR_IN
-Text GLabel 7850 3650 0    39   Input ~ 0
-SolarPWR_OUT
 $Comp
 L GND #PWR016
@@
 Text Notes 10650 7650 2    39   ~ 0
 1
+Text GLabel 7850 3650 0    39   Input ~ 0
+SolarPWR_IN
 $EndSCHEMATC

Commit message: added gerbers
Parts:
- J11, J13: footprint Connectors_Molex:Molex_NanoFit_1x02x2.50mm_Straight -> Pin_Headers:Pin_Header_Straight_1x02_Pitch2.54mm
Changed lines of the file:
@@
 F 0 "J11" H 7100 3750 50  0000 C CNN
 F 1 "Conn_01x02_Female" H 7100 3450 50  0000 C CNN
-F 2 "Connectors_Molex:Molex_NanoFit_1x02x2.50mm_Straight" H 7100 3650 50  0001 C CNN
+F 2 "Pin_Headers:Pin_Header_Straight_1x02_Pitch2.54mm" H 7100 3650 50  0001 C CNN
 F 3 "" H 7100 3650 50  0001 C CNN
 	1    7100 3650
@@
 F 0 "J13" H 8150 3750 50  0000 C CNN
 F 1 "Conn_01x02_Female" H 8150 3450 50  0000 C CNN
-F 2 "Connectors_Molex:Molex_NanoFit_1x02x2.50mm_Straight" H 8150 3650 50  0001 C CNN
+F 2 "Pin_Headers:Pin_Header_Straight_1x02_Pitch2.54mm" H 8150 3650 50  0001 C CNN
 F 3 "" H 8150 3650 50  0001 C CNN
 F 4 "105309-1102" H 8150 3650 60  0001 C CNN "P#"
